File: esp_lights_on.kicad_pcb (KiCad board)
At the start: 2 copper layers, 50.7 x 58.5 mm, 14 parts, among them J1 Conn_01x04_Pin, J2 VOUT, J3 VIN, K1 RELAY, Q1 SS8050, U1 ESP32-WROOM-32, U2 TLV1117-33

Commit message: commit non-verified
Routing:
- net VOUT_5V: track 0.00 -> 69.3 mm, vias 0 -> 2
- net VIN_NULL: track 0.00 -> 57.6 mm, vias 0 -> 1
- net VIN_220V: track 0.00 -> 44.6 mm
- net +3.3V: track 0.00 -> 33.6 mm
- net RX: track 0.00 -> 27.7 mm, vias 0 -> 3
- net TX: track 0.00 -> 22.0 mm, vias 0 -> 1
- net VOUT_220V: track 0.00 -> 11.0 mm
- net SW: track 0.00 -> 10.2 mm
- net COLECTOR: track 0.00 -> 8.79 mm, vias 1 -> 0
- net GND: vias 0 -> 11

Commit message: some commits
Routing:
- net VIN_NULL: track 57.6 -> 20.4 mm, vias 1 -> 0
- net VOUT_5V: track 69.3 -> 67.8 mm
Changed lines of the file:
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@@
 		(net "+3.3V")
+	)
+	(gr_poly
+		(pts
+			(xy 128.848513 109.368265) (xy 128.75 105.1) (xy 168.69 105.4) (xy 170.23 104.07) (xy 173.32 104.07)
+			(xy 173.350073 109.102323)
+		)
+		(stroke
+			(width 0.2)
+			(type solid)
+		)
+		(fill yes)
+		(layer "B.Cu")
+		(net "VIN_NULL")
 	)
 	(gr_rect
@@
 	)
 	(segment
-		(start 141.77 100.98)
-		(end 141.77 100.5925)
-		(width 1)
-		(layer "F.Cu")
-		(net "VIN_NULL")
-	)
-	(segment
-		(start 141.77 100.5925)
+		(start 131.3275 96.6725)
 		(end 137.85 96.6725)
 		(width 1)
-		(layer "F.Cu")
-		(net "VIN_NULL")
-	)
-	(via
-		(at 141.77 100.98)
-		(size 1.3)
-		(drill 0.7)
-		(layers "F.Cu" "B.Cu")
-		(net "VIN_NULL")
-	)
-	(segment
-		(start 127.57 100.63)
-		(end 131.5275 96.6725)
-		(width 1)
-		(layer "B.Cu")
-		(net "VIN_NULL")
-	)
-	(segment
-		(start 171.0325 106.465)
-		(end 147.255 106.465)
+		(layer "B.Cu")
+		(net "VIN_NULL")
+	)
+	(segment
+		(start 127.42 104.72)
+		(end 127.42 100.58)
+		(width 1)
+		(layer "B.Cu")
+		(net "VIN_NULL")
+	)
+	(segment
+		(start 127.42 100.58)
+		(end 131.3275 96.6725)
 		(width 1)
 		(layer "B.Cu")
@@
 	(segment
 		(start 130.39 107.69)
-		(end 127.57 104.87)
-		(width 1)
-		(layer "B.Cu")
-		(net "VIN_NULL")
-	)
-	(segment
-		(start 127.57 104.87)
-		(end 127.57 100.63)
-		(width 1)
-		(layer "B.Cu")
-		(net "VIN_NULL")
-	)
-	(segment
-		(start 147.255 106.465)
-		(end 141.77 100.98)
-		(width 1)
-		(layer "B.Cu")
-		(net "VIN_NULL")
-	)
-	(segment
-		(start 131.5275 96.6725)
-		(end 137.85 96.6725)
+		(end 127.42 104.72)
 		(width 1)
 		(layer "B.Cu")
@@
 		(drill 0.7)
 		(layers "F.Cu" "B.Cu")
-		(net "VOUT_5V")
-	)
-	(segment
-		(start 164.7 81.41)
-		(end 165.19 80.92)
-		(width 0.5)
-		(layer "B.Cu")
 		(net "VOUT_5V")
 	)
@@
 	)
 	(segment
-		(start 137.85 76.3525)
-		(end 142.9075 81.41)
-		(width 0.5)
-		(layer "B.Cu")
-		(net "VOUT_5V")
-	)
-	(segment
-		(start 165.19 80.92)
-		(end 166.3275 80.92)
+		(start 167.7475 79.5)
+		(end 169.5875 77.66)
 		(width 0.5)
 		(layer "B.Cu")
@@
 	)
 	(segment
+		(start 145.07 79.5)
+		(end 167.7475 79.5)
+		(width 0.5)
+		(layer "B.Cu")
+		(net "VOUT_5V")
+	)
+	(segment
 		(start 135.465 76.3525)
 		(end 127.42 68.3075)
@@
 	)
 	(segment
-		(start 166.3275 80.92)
-		(end 169.5875 77.66)
-		(width 0.5)
-		(layer "B.Cu")
-		(net "VOUT_5V")
-	)
-	(segment
-		(start 142.9075 81.41)
-		(end 164.7 81.41)
+		(start 137.85 76.3525)
+		(end 141.9225 76.3525)
 		(width 0.5)
 		(layer "B.Cu")
@@
 		(width 0.5)
 		(layer "B.Cu")
+		(net "VOUT_5V")
+	)
+	(segment
+		(start 141.9225 76.3525)
+		(end 145.07 79.5)
+		(width 0.5)
+		(layer "B.Cu")

Commit message: some other updates unverified
Parts:
- removed J1: Conn_01x04_Pin, Connector_PinHeader_2.54mm:PinHeader_1x04_P2.54mm_Vertical
- added D2: D, Diode_SMD:D_SMA_Handsoldering, B.Cu at (196.9, 37.3)
- added F1: Fuse_Small, Fuse:Fuse_Schurter_UMZ250, B.Cu at (201.8, 72.4)
- added J4: Screw_Terminal_01x03, TerminalBlock_Phoenix:TerminalBlock_Phoenix_MKDS-1,5-3-5.08_1x03_P5.08mm_Horizontal, F.Cu at (221.1, 85.9)
- added K2: RELAY, Relay_THT:Relay_SPST_Panasonic_ADW11, F.Cu at (225.0, 57.0)
- added Q2: SS8050, Package_TO_SOT_SMD:SOT-23-3, B.Cu at (192.0, 34.8)
- added R2: 1k, Resistor_SMD:R_1206_3216Metric_Pad1.30x1.75mm_HandSolder, B.Cu at (190.9, 39.9)
- D1, Q1: moved to F.Cu
- J2: value VOUT -> Conn_01x06_Pin; footprint TerminalBlock_Phoenix:TerminalBlock_Phoenix_MKDS-1,5-2-5.08_1x02_P5.08mm_Horizontal -> Connector_PinHeader_2.54mm:PinHeader_1x06_P2.54mm_Vertical
- moved J2 97.0 mm to (237.3, 35.6), turned to 0 degrees
- moved C3 77.8 mm to (206.1, 35.8)
- moved C2 77.7 mm to (208.2, 35.7)
- moved C4 77.6 mm to (204.0, 35.8)
- moved U2 76.7 mm to (204.1, 44.2)
- moved U1 68.9 mm to (219.7, 41.4)
- moved K1 67.6 mm to (235.9, 56.8)
- moved J3 67.3 mm to (194.8, 83.0)
- moved PS1 58.2 mm to (202.7, 66.6)
- moved D1 41.8 mm to (197.8, 49.3), turned to 90 degrees
- moved Q1 33.8 mm to (192.1, 47.5), turned to 0 degrees
- moved R1 33.5 mm to (191.0, 43.0)
- moved C1 25.1 mm to (192.6, 51.3), turned to 90 degrees
Connections:
- net COLECTOR renamed COLECTOR1
- net SW renamed SW1
- J2 pad 1: VIN_NULL -> VOUT_5V
- J2 pad 2: VOUT_220V -> RX
- J3 pad 2: VIN_NULL -> NULL
- K1 pad 14: VOUT_220V -> circuit1
- PS1 pad 1: VIN_220V -> VIN_220V_traf
- PS1 pad 2: VIN_NULL -> NULL
- U1 pad 25: unconnected-(U1-IO0-Pad25) -> BOOt
- U1 pad 3: unconnected-(U1-EN-Pad3) -> EN
- U1 pad 31: unconnected-(U1-IO19-Pad31) -> SW2
Routing:
- net COLECTOR2: track 0.00 -> 43.1 mm, vias 0 -> 2
- net NULL: track 0.00 -> 42.1 mm
- net SW2: track 0.00 -> 39.4 mm, vias 0 -> 1
- net SW1: track 10.2 -> 45.1 mm, vias 0 -> 2
- net COLECTOR1: track 8.79 -> 40.3 mm, vias 0 -> 1
- net EN: track 0.00 -> 30.5 mm, vias 0 -> 2
- net VOUT_5V: track 67.8 -> 95.5 mm, vias 2 -> 5
- net VIN_NULL: track 20.4 -> 0.00 mm
- net RX: track 27.7 -> 9.42 mm, vias 3 -> 1
- net circuit2: track 0.00 -> 13.3 mm
- net BOOt: track 0.00 -> 12.5 mm
- net TX: track 22.0 -> 9.85 mm
- net VOUT_220V: track 11.0 -> 0.00 mm
- net circuit1: track 0.00 -> 9.34 mm
- net VIN_220V: track 44.6 -> 53.0 mm
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Other:
- board size 50.7 x 58.5 mm -> 50 x 60 mm

Commit message: final commit
Parts:
- C1, D1: moved to B.Cu
- R1, R2: footprint Resistor_SMD:R_1206_3216Metric_Pad1.30x1.75mm_HandSolder -> Resistor_SMD:R_0805_2012Metric
- moved D1 36.0 mm to (232.3, 59.5), turned to 180 degrees
- moved D2 32.8 mm to (221.2, 59.3), turned to 180 degrees
- moved C2 13.1 mm to (207.3, 48.8)
- moved R2 8.76 mm to (199.5, 41.6), turned to 180 degrees
- moved Q2 8.24 mm to (199.7, 37.8)
- moved C1 7.16 mm to (197.9, 56.2), turned to 0 degrees
- moved J3 4.45 mm to (199.2, 83.0)
- moved J2 3.18 mm to (235.4, 38.2)
- moved R1 2.80 mm to (193.4, 44.4)
- moved Q1 2.40 mm to (193.8, 49.2)
- moved C4 2.14 mm to (206.1, 35.4)
- moved C3 2.12 mm to (208.2, 35.4)
Connections:
- C2 pad 2: Net-(C2-Pad2) -> GND
- C3 pad 2: Net-(C2-Pad2) -> GND
Routing:
- net SW2: track 39.4 -> 33.8 mm
- net EN: track 30.5 -> 34.7 mm, vias 2 -> 1
- net VIN_220V: track 53.0 -> 49.4 mm
- net COLECTOR2: track 43.1 -> 46.4 mm, vias 2 -> 0
- net COLECTOR1: track 40.3 -> 42.7 mm
- net NULL: track 42.1 -> 39.8 mm
- net BOOt: track 12.5 -> 10.6 mm, vias 0 -> 1
- net +3.3V: track 28.2 -> 29.8 mm
- net Net-(Q1-B): track 1.98 -> 3.24 mm
- net VOUT_5V: track 95.5 -> 95.4 mm, vias 5 -> 4
- net GND: vias 7 -> 5
Other:
- outline, holes or cut-outs redrawn

Commit message: fixes
Routing:
- net circuit1: track 9.34 -> 15.9 mm
- net circuit2: track 13.3 -> 18.0 mm
- net VIN_220V: track 49.4 -> 47.2 mm
Other:
- outline, holes or cut-outs redrawn

Commit message: other fixes
Parts:
- moved K2 2.01 mm to (226.2, 55.4)
Routing:
- net COLECTOR2: track 46.4 -> 35.3 mm
- net circuit2: track 18.0 -> 17.4 mm
- net circuit1: track 15.9 -> 15.3 mm

Commit message: some other fixes
Parts:
- moved K2 20.9 mm to (216.1, 73.7), turned to 90 degrees
- moved K1 19.0 mm to (227.0, 73.5), turned to 90 degrees
- turned D1 to 0 degrees
- turned D2 to 0 degrees
Routing:
- net COLECTOR2: track 35.3 -> 52.9 mm, vias 0 -> 2
- net COLECTOR1: track 42.7 -> 50.0 mm
- net VIN_220V: track 47.0 -> 39.8 mm
- net circuit2: track 17.4 -> 14.3 mm
- net VOUT_5V: track 95.3 -> 96.6 mm, vias 4 -> 5
- net circuit1: track 15.3 -> 16.1 mm
