File: esp_lights_on.kicad_sch (KiCad schematic)
At the start: 0 parts

Commit message: some commits
Parts:
- added C1: 10uF, Capacitor_SMD:C_1210_3225Metric_Pad1.33x2.70mm_HandSolder, symbol Device:C
- added C2: 10uF, Capacitor_SMD:C_0805_2012Metric_Pad1.18x1.45mm_HandSolder, symbol Device:C
- added C3, C4: 100nF, Capacitor_SMD:C_0805_2012Metric_Pad1.18x1.45mm_HandSolder, symbol Device:C
- added D1: D, Diode_SMD:D_SMA_Handsoldering, symbol Device:D
- added J1: Conn_01x04_Pin, Connector_PinHeader_2.54mm:PinHeader_1x04_P2.54mm_Vertical, symbol Connector:Conn_01x04_Pin
- added J2: VOUT, TerminalBlock_Phoenix:TerminalBlock_Phoenix_MKDS-1,5-2-5.08_1x02_P5.08mm_Horizontal, symbol Connector:Screw_Terminal_01x02
- added J3: VIN, TerminalBlock_Phoenix:TerminalBlock_Phoenix_MKDS-1,5-2-5.08_1x02_P5.08mm_Horizontal, symbol Connector:Screw_Terminal_01x02
- added K1: RELAY, Relay_THT:Relay_SPST_Panasonic_ADW11, symbol Relay:ADW11
- added PS1: POWER, RACM06E-12SK_277:CONV_RACM06E-12SK_277, symbol RACM06E-12SK_277:RACM06E-12SK_277
- added Q1: SS8050, Package_TO_SOT_SMD:SOT-23-3, symbol Transistor_BJT:SS8050
- added R1: 1k, Resistor_SMD:R_1206_3216Metric_Pad1.30x1.75mm_HandSolder, symbol Device:R
- added U1: ESP32-WROOM-32, RF_Module:ESP32-WROOM-32, symbol RF_Module:ESP32-WROOM-32
- added U2: TLV1117-33, Package_TO_SOT_SMD:SOT-223-3_TabPin2, symbol Regulator_Linear:TLV1117-33
Connections:
- new net: Q1.1 (B), R1.2
- new net: C2.2, C3.2
- new net +3.3V: C2.1, C3.1, C4.1, U1.2 (VDD), U2.2 (VO)
- new net COLECTOR: D1.2 (A), K1.A2, Q1.3 (C)
- new net GND: C1.2, C4.2, J1.4 (Pin_4), PS1.4 (-VOUT), Q1.2 (E), U1.1 (GND), U1.15 (GND), U1.38 (GND), U1.39 (GND), U2.1 (GND)
- new net RX: J1.2 (Pin_2), U1.35 (TXD0/IO1)
- new net SW: R1.1, U1.33 (IO21)
- new net TX: J1.3 (Pin_3), U1.34 (RXD0/IO3)
- new net VIN_220V: J3.1 (Pin_1), K1.13, PS1.1 (VAC_IN(L))
- new net VIN_NULL: J2.1 (Pin_1), J3.2 (Pin_2), PS1.2 (VAC_IN(N))
- new net VOUT_220V: J2.2 (Pin_2), K1.14
- new net VOUT_5V: C1.1, D1.1 (K), J1.1 (Pin_1), K1.A1, PS1.5 (+VOUT), U2.3 (VI)

Commit message: modification by ovi
Parts:
- added F1: Fuse_Small, Fuse:Fuse_Schurter_UMZ250, symbol Device:Fuse_Small
Connections:
- net VIN_220V: now also F1.2; no longer J3.1 (Pin_1)
- new net: F1.1, J3.1 (Pin_1)
Other:
- moved on the sheet: C4, J3, PS1, U1

Commit message: some other updates unverified
Parts:
- removed J1: Conn_01x04_Pin, Connector_PinHeader_2.54mm:PinHeader_1x04_P2.54mm_Vertical, symbol Connector:Conn_01x04_Pin
- removed J2: VOUT, TerminalBlock_Phoenix:TerminalBlock_Phoenix_MKDS-1,5-2-5.08_1x02_P5.08mm_Horizontal, symbol Connector:Screw_Terminal_01x02
- added D2: D, Diode_SMD:D_SMA_Handsoldering, symbol Device:D
- added J2: Conn_01x06_Pin, Connector_PinHeader_2.54mm:PinHeader_1x06_P2.54mm_Vertical, symbol Connector:Conn_01x06_Pin
- added J4: Screw_Terminal_01x03, TerminalBlock_Phoenix:TerminalBlock_Phoenix_MKDS-1,5-3-5.08_1x03_P5.08mm_Horizontal, symbol Connector:Screw_Terminal_01x03
- added K2: RELAY, Relay_THT:Relay_SPST_Panasonic_ADW11, symbol Relay:ADW11
- added Q2: SS8050, Package_TO_SOT_SMD:SOT-23-3, symbol Transistor_BJT:SS8050
- added R2: 1k, Resistor_SMD:R_1206_3216Metric_Pad1.30x1.75mm_HandSolder, symbol Device:R
Connections:
- net GND: now also J2.6 (Pin_6), Q2.2 (E)
- net RX: now also J2.2 (Pin_2)
- net TX: now also J2.3 (Pin_3)
- net VIN_220V: now also F1.1, J3.1 (Pin_1), K2.13; no longer F1.2, PS1.1 (VAC_IN(L))
- net VOUT_5V: now also D2.1 (K), J2.1 (Pin_1), K2.A1
- net BOOt: now reaches U1.25 (IO0)
- net BOOt: now also J2.4 (Pin_4)
- net EN: now reaches U1.3 (EN)
- net EN: now also J2.5 (Pin_5)
- net SW2: now reaches U1.31 (IO19)
- net SW2: now also R2.1
- net COLECTOR renamed COLECTOR1
- net SW renamed SW1
- net VIN_NULL renamed NULL
- net NULL: now also J4.1 (Pin_1)
- net VOUT_220V renamed circuit1
- net circuit1: now also J4.3 (Pin_3)
- new net: Q2.1 (B), R2.2
- new net COLECTOR2: D2.2 (A), K2.A2, Q2.3 (C)
- new net VIN_220V_traf: F1.2, PS1.1 (VAC_IN(L))
- new net circuit2: J4.2 (Pin_2), K2.14
Other:
- moved on the sheet: C1, C4, D1, F1, J3, K1, PS1, Q1, R1, U1

Commit message: final commit
Parts:
- R1, R2: footprint Resistor_SMD:R_1206_3216Metric_Pad1.30x1.75mm_HandSolder -> Resistor_SMD:R_0805_2012Metric
Connections:
- net GND: now also C2.2, C3.2
Other:
- moved on the sheet: C3
Changed lines of the file:
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@@
 	)
 	(junction
-		(at 173.99 96.52)
+		(at 106.68 45.72)
 		(diameter 0)
 		(color 0 0 0 0)
 	)
 	(junction
-		(at 127 35.56)
+		(at 173.99 96.52)
 		(diameter 0)
 		(color 0 0 0 0)
@@
 	)
 	(junction
+		(at 115.57 45.72)
+		(diameter 0)
+		(color 0 0 0 0)
+	)
+	(junction
 		(at 250.19 96.52)
 		(diameter 0)
@@
 	)
 	(junction
-		(at 115.57 43.18)
+		(at 127 35.56)
 		(diameter 0)
 		(color 0 0 0 0)
@@
 	(wire
 		(pts
-			(xy 106.68 43.18) (xy 115.57 43.18)
+			(xy 106.68 45.72) (xy 115.57 45.72)
 		)
 		(stroke
@@
 	(wire
 		(pts
+			(xy 115.57 45.72) (xy 127 45.72)
+		)
+		(stroke
+			(width 0)
+			(type default)
+		)
+	)
+	(wire
+		(pts
 			(xy 95.25 63.5) (xy 95.25 64.77)
 		)
@@
 	(wire
 		(pts
+			(xy 127 36.83) (xy 127 35.56)
+		)
+		(stroke
+			(width 0)
+			(type default)
+		)
+	)
+	(wire
+		(pts
 			(xy 173.99 96.52) (xy 177.8 96.52)
 		)
@@
 	(wire
 		(pts
-			(xy 182.88 114.3) (xy 182.88 111.76)
+			(xy 115.57 45.72) (xy 115.57 43.18)
 		)
 		(stroke
@@
 	(wire
 		(pts
-			(xy 83.82 142.24) (xy 88.9 142.24)
+			(xy 182.88 114.3) (xy 182.88 111.76)
 		)
 		(stroke
@@
 	(wire
 		(pts
-			(xy 93.98 34.29) (xy 99.06 34.29)
+			(xy 83.82 142.24) (xy 88.9 142.24)
 		)
 		(stroke
@@
 	(wire
 		(pts
-			(xy 252.73 96.52) (xy 252.73 97.79)
+			(xy 93.98 34.29) (xy 99.06 34.29)
 		)
 		(stroke
@@
 	(wire
 		(pts
-			(xy 102.87 58.42) (xy 102.87 69.85)
+			(xy 252.73 96.52) (xy 252.73 97.79)
 		)
 		(stroke
@@
 	(wire
 		(pts
-			(xy 220.98 78.74) (xy 218.44 78.74)
+			(xy 102.87 58.42) (xy 102.87 69.85)
 		)
 		(stroke
@@
 	(wire
 		(pts
-			(xy 115.57 43.18) (xy 127 43.18)
+			(xy 220.98 78.74) (xy 218.44 78.74)
 		)
 		(stroke
@@
 	(wire
 		(pts
+			(xy 106.68 45.72) (xy 106.68 46.99)
+		)
+		(stroke
+			(width 0)
+			(type default)
+		)
+	)
+	(wire
+		(pts
 			(xy 250.19 116.84) (xy 250.19 96.52)
 		)
@@
 	(wire
 		(pts
+			(xy 106.68 41.91) (xy 106.68 45.72)
+		)
+		(stroke
+			(width 0)
+			(type default)
+		)
+	)
+	(wire
+		(pts
 			(xy 146.05 30.48) (xy 146.05 34.29)
 		)
@@
 	(wire
 		(pts
-			(xy 120.65 34.29) (xy 114.3 34.29)
+			(xy 127 45.72) (xy 127 44.45)
 		)
 		(stroke
@@
 	(wire
 		(pts
-			(xy 104.14 119.38) (xy 104.14 132.08)
+			(xy 120.65 34.29) (xy 114.3 34.29)
 		)
 		(stroke
@@
 	(wire
 		(pts
-			(xy 100.33 119.38) (xy 104.14 119.38)
+			(xy 104.14 119.38) (xy 104.14 132.08)
 		)
 		(stroke
@@
 	(wire
 		(pts
-			(xy 106.68 41.91) (xy 106.68 44.45)
+			(xy 100.33 119.38) (xy 104.14 119.38)
 		)
 		(stroke
@@
 			)
 		)
-		(property "Footprint" "Resistor_SMD:R_1206_3216Metric_Pad1.30x1.75mm_HandSolder"
+		(property "Footprint" "Resistor_SMD:R_0805_2012Metric"
 			(at 93.472 68.58 90)
 			(hide yes)
@@
 	(symbol
 		(lib_id "Device:C")
-		(at 127 39.37 0)
+		(at 127 40.64 0)
 		(unit 1)
 		(body_style 1)
@@
 		(fields_autoplaced yes)
 		(property "Reference" "C3"
-			(at 130.81 38.0999 0)
+			(at 130.81 39.3699 0)
 			(show_name no)
 			(do_not_autoplace no)
@@
 		)
 		(property "Value" "100nF"
-			(at 130.81 40.6399 0)
+			(at 130.81 41.9099 0)
 			(show_name no)
 			(do_not_autoplace no)
@@
 		)
 		(property "Footprint" "Capacitor_SMD:C_0805_2012Metric_Pad1.18x1.45mm_HandSolder"
-			(at 127.9652 43.18 0)
+			(at 127.9652 44.45 0)
 			(hide yes)
 			(show_name no)
@@
 		)
 		(property "Datasheet" ""
-			(at 127 39.37 0)
+			(at 127 40.64 0)
 			(hide yes)
 			(show_name no)
@@
 		)
 		(property "Description" "Unpolarized capacitor"
-			(at 127 39.37 0)
+			(at 127 40.64 0)
 			(hide yes)
 			(show_name no)
@@
 	(symbol
 		(lib_id "power:GND")
-		(at 106.68 44.45 0)
+		(at 106.68 46.99 0)
 		(unit 1)
 		(body_style 1)
@@
 		(fields_autoplaced yes)
 		(property "Reference" "#PWR01"
-			(at 106.68 50.8 0)
+			(at 106.68 53.34 0)
 			(hide yes)
 			(show_name no)
@@
 		)
 		(property "Value" "GND"
-			(at 106.68 49.53 0)
+			(at 106.68 52.07 0)
 			(show_name no)
 			(do_not_autoplace no)
@@
 		)
 		(property "Footprint" ""
-			(at 106.68 44.45 0)
+			(at 106.68 46.99 0)
 			(hide yes)
 			(show_name no)
@@
 		)
 		(property "Datasheet" ""
-			(at 106.68 44.45 0)
+			(at 106.68 46.99 0)
 			(hide yes)
 			(show_name no)
@@
 		)
 		(property "Description" "Power symbol creates a global label with name \"GND\" , ground"
-			(at 106.68 44.45 0)
+			(at 106.68 46.99 0)
 			(hide yes)
 			(show_name no)
@@
 			)
 		)
-		(property "Footprint" "Resistor_SMD:R_1206_3216Metric_Pad1.30x1.75mm_HandSolder"
+		(property "Footprint" "Resistor_SMD:R_0805_2012Metric"
 			(at 125.222 69.85 90)
 			(hide yes)

Commit message: modifications by ovi
Parts:
- K1, K2: footprint Relay_THT:Relay_SPST_Panasonic_ADW11 -> RELAYs:0JT-SS-105LM
Changed lines of the file:
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@@
 			)
 		)
-		(property "Footprint" "Relay_THT:Relay_SPST_Panasonic_ADW11"
+		(property "Footprint" "RELAYs:0JT-SS-105LM"
 			(at 45.72 146.05 0)
 			(hide yes)
@@
 			)
 		)
-		(property "Footprint" "Relay_THT:Relay_SPST_Panasonic_ADW11"
+		(property "Footprint" "RELAYs:0JT-SS-105LM"
 			(at 95.25 148.59 0)
 			(hide yes)
